File: bbb-parallel-cape.kicad_pcb (KiCad board)
At the start: 2 copper layers, 54.6 x 86.4 mm, 45 parts, among them IC201 GTL2003PW, IC202 GTL2003PW, IC203 GTL2003PW, IC204 GTL2003PW, IC205 GTL2003PW, P101 IDC26, P102 BeagleBone_Black_Header, P103 BeagleBone_Black_Header, P104 IDC26, P105 Conn_02x03_Odd_Even, Q101 2N7002K, SW101 SW_Push, SW102 SW_Push

Commit message: before edge cut
Parts:
- Z105: footprint footprint:515-1114F -> footprint:515-1114F_2
- moved RN209 138.5 mm to (128.2, 81.8), turned to 180 degrees
- moved IC205 129.3 mm to (127.3, 88.5), turned to 270 degrees
- moved R210 125.8 mm to (133.4, 92.7), turned to 90 degrees
- moved C205 121.8 mm to (133.4, 88.5), turned to 90 degrees
- moved R209 118.8 mm to (133.4, 84.1), turned to 270 degrees
- moved RN205 113.6 mm to (129.1, 51.0), turned to 180 degrees
- moved RN208 112.6 mm to (143.4, 81.8), turned to 180 degrees
- moved RN207 110.0 mm to (139.2, 81.8), turned to 180 degrees
- moved R102 99.2 mm to (156.9, 125.3), turned to 180 degrees
- moved IC204 98.1 mm to (141.1, 88.5), turned to 270 degrees
- moved R212 96.0 mm to (122.8, 114.2), turned to 270 degrees
- moved IC202 94.5 mm to (131.2, 57.5), turned to 270 degrees
- moved R208 93.8 mm to (147.2, 92.7), turned to 90 degrees
- moved R101 93.7 mm to (156.9, 117.6), turned to 180 degrees
- moved R211 92.2 mm to (122.8, 110.2), turned to 270 degrees
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Other:
- outline, holes or cut-outs redrawn
- net class Big added: clearance 0.1778, trace_width 0.3048, via_dia 0.6, via_drill 0.4
- net class Default: clearance 0.2 -> 0.1778; trace_width 0.25 -> 0.1778
- net class Output added: clearance 0.1778, trace_width 0.254, via_dia 0.6, via_drill 0.4
- net class Power added: clearance 0.1778, trace_width 0.381, via_dia 0.6, via_drill 0.4
- rule trace_clearance: 0.2 -> 0.1778
- rule trace_min: 0.2 -> 0.1778

Commit message: revision1 files
Parts:
- added G***: LOGO, footprint:OSHW, F.Cu at (140.6, 69.6)
- moved SW102 74.1 mm to (129.8, 51.4), turned to 270 degrees
- moved SW101 73.9 mm to (120.8, 51.2), turned to 90 degrees
- moved RN204 20.7 mm to (149.8, 71.5), turned to 270 degrees
- moved RN201 16.4 mm to (149.8, 67.0), turned to 270 degrees
- moved IC201 13.4 mm to (156.3, 69.2), turned to 0 degrees
- moved IC202 11.5 mm to (126.2, 68.0)
- moved RN205 11.5 mm to (124.0, 61.4)
- moved RN202 11.5 mm to (128.4, 61.4)
- moved C202 11.5 mm to (132.4, 67.7)
- moved R203 11.5 mm to (132.4, 63.5)
- moved R204 11.5 mm to (132.3, 72.2)
- moved R211 11.0 mm to (122.8, 121.2)
- moved R212 11.0 mm to (122.8, 125.2)
- moved P101 9.75 mm to (141.8, 81.0)
- moved R206 8.80 mm to (160.6, 101.4)
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Routing:
- net GNDD: track 0.00 -> 1074.0 mm, vias 0 -> 166
- net SYS_5V: track 0.00 -> 200.2 mm, vias 0 -> 2
- net PU_OR_PD: track 0.00 -> 189.3 mm, vias 0 -> 2
- net +3V3: track 0.00 -> 107.7 mm, vias 0 -> 1
- net SYS_RESETn: track 0.00 -> 105.9 mm
- net PWR_BUT: track 0.00 -> 103.7 mm, vias 0 -> 1
- net IO5_BB: track 0.00 -> 92.3 mm, vias 0 -> 1
- net GND_OR_5V: track 0.00 -> 77.4 mm
- net IO15_BB: track 0.00 -> 64.3 mm, vias 0 -> 2
- net IO1_BB: track 0.00 -> 58.4 mm, vias 0 -> 2
- net IO8_BB: track 0.00 -> 58.2 mm, vias 0 -> 1
- net IO19_BB: track 0.00 -> 56.4 mm, vias 0 -> 1
- net IO3_BB: track 0.00 -> 54.5 mm, vias 0 -> 1
- net IO16_BB: track 0.00 -> 52.6 mm, vias 0 -> 1
- net IO17_BB: track 0.00 -> 51.8 mm, vias 0 -> 2
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- added copper zone on B.Cu, net GNDD
- added copper zone on F.Cu, net GNDD
Other:
- outline, holes or cut-outs redrawn
- board text added: "Parallel Cape Revision 1"

Commit message: revision 1.1 before via stitching
Parts:
- Q101: footprint 2N7002K-7:SOT95P240X105-3N -> footprint:SOT95P240X105-3N
- moved Z106 93.1 mm to (162.0, 42.7), turned to 180 degrees
- moved D2 74.6 mm to (160.5, 51.9), turned to 180 degrees
- moved R102 74.0 mm to (155.7, 52.1), turned to 0 degrees
- moved Q101 66.4 mm to (166.0, 55.4), turned to 180 degrees
- moved P105 62.9 mm to (129.0, 61.0), turned to 90 degrees
- moved D1 59.5 mm to (160.5, 59.4), turned to 180 degrees
- moved R101 58.6 mm to (155.7, 59.8), turned to 0 degrees
- moved R201 46.6 mm to (123.8, 94.1), turned to 90 degrees
- moved R202 42.5 mm to (123.8, 85.3), turned to 270 degrees
- moved JP101 42.1 mm to (156.0, 90.2)
- moved C201 41.4 mm to (123.8, 89.9), turned to 270 degrees
- moved RN207 33.6 mm to (135.0, 123.8), turned to 0 degrees
- moved RN208 33.4 mm to (142.5, 123.8), turned to 0 degrees
- moved RN209 33.4 mm to (128.8, 123.8), turned to 0 degrees
- moved RN206 33.3 mm to (149.5, 123.8), turned to 0 degrees
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- renumbered Z105 to Z106
Connections:
- net PU_OR_PD renamed PULLUP_REF
- JP101 pad 6: GNDD -> +3V3
- RN201 pad 5: IO3_BB -> IO0
- RN201 pad 6: IO2_BB -> IO1
- RN201 pad 7: IO1_BB -> IO2
- RN201 pad 8: IO0_BB -> IO3
- RN202 pad 5: IO11_BB -> IO8
- RN202 pad 6: IO10_BB -> IO9
- RN202 pad 7: IO9_BB -> IO10
- RN202 pad 8: IO8_BB -> IO11
- RN203 pad 5: IO19_BB -> IO16
- RN203 pad 6: IO18_BB -> IO17
- RN203 pad 7: IO17_BB -> IO18
- RN203 pad 8: IO16_BB -> IO19
- RN204 pad 5: IO7_BB -> IO4
- RN204 pad 6: IO6_BB -> IO5
- RN204 pad 7: IO5_BB -> IO6
- RN204 pad 8: IO4_BB -> IO7
- RN205 pad 5: IO15_BB -> IO12
- RN205 pad 6: IO14_BB -> IO13
- RN205 pad 7: IO13_BB -> IO14
- RN205 pad 8: IO12_BB -> IO15
- RN206 pad 5: IO23_BB -> IO20
- RN206 pad 6: IO22_BB -> IO21
- RN206 pad 7: IO21_BB -> IO22
- RN206 pad 8: IO20_BB -> IO23
- RN207 pad 5: IO31_BB -> IO28
- RN207 pad 6: IO30_BB -> IO29
- RN207 pad 7: IO29_BB -> IO30
- RN207 pad 8: IO28_BB -> IO31
- RN208 pad 5: IO27_BB -> IO24
- RN208 pad 6: IO26_BB -> IO25
- RN208 pad 7: IO25_BB -> IO26
- RN208 pad 8: IO24_BB -> IO27
- RN209 pad 7: IO33_BB -> IO32
- RN209 pad 8: IO32_BB -> IO33
Routing:
- net GNDD: track 1074.0 -> 0.00 mm, vias 166 -> 0
- net SYS_RESETn: track 105.9 -> 36.8 mm
- net IO5_BB: track 92.3 -> 37.3 mm, vias 1 -> 2
- net PWR_BUT: track 103.7 -> 48.8 mm
- net PULLUP_REF: track 189.3 -> 135.5 mm
- net IO1_BB: track 58.4 -> 12.8 mm, vias 2 -> 1
- net IO15_BB: track 64.3 -> 20.2 mm, vias 2 -> 1
- net IO3_BB: track 54.5 -> 17.7 mm, vias 1 -> 2
- net IO2_BB: track 17.9 -> 45.7 mm
- net IO8_BB: track 58.2 -> 30.4 mm
- net +3V3: track 107.7 -> 80.3 mm, vias 1 -> 0
- net IO4_BB: track 18.7 -> 44.1 mm
- net IO19_BB: track 56.4 -> 80.1 mm, vias 1 -> 3
- net IO6_BB: track 17.8 -> 41.1 mm
- net GND_OR_5V: track 77.4 -> 98.5 mm, vias 0 -> 6
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Other:
- board size 54.6 x 86.4 mm -> 66.7 x 86.4 mm
- board text added: "1"
- board text added: "10"
- board text added: "11"
- board text added: "12"
- board text added: "13"
- board text added: "14"
- board text added: "15"
- board text added: "16"
- board text added: "17"
- board text added: "18"
- board text added: "19"
- board text added: "2"
- board text added: "20"
- board text added: "21"
- board text added: "22"
- board text added: "23"
- board text added: "24"
- board text added: "25"
- board text added: "26"
- board text added: "27"
- board text added: "28"
- board text added: "29"
- board text added: "3"
- board text added: "30"
- board text added: "31"
- board text added: "32"
- board text added: "33"
- board text added: "3V3"
- board text added: "4"
- board text added: "5"
- board text added: "5V"
- board text added: "6"
- board text added: "7"
- board text added: "8"
- board text added: "9"
- board text added: "GND"
- board text added: "OUT"
- board text added: "PU"
- board text added: "PWR"
- board text added: "Parallel Cape by Alexander Rössler"
- board text added: "RST"
- board text added: "Rev 1.1"
- board text removed: "Parallel Cape Revision 1"

Commit message: completing Rev 1.1
Routing:
- net GNDD: track 0.00 -> 1034.0 mm, vias 0 -> 211
- net (no net): track 0.00 -> 13.6 mm, vias 0 -> 2
- net PULLUP_REF: track 135.5 -> 142.9 mm
- net Net-(IC205-Pad2): track 4.67 -> 8.14 mm
- net GND_OR_5V: track 98.5 -> 99.5 mm
- net Net-(C201-Pad1): track 9.30 -> 10.3 mm

Commit message: updating project
Other:
- board text added: "0"
- board text added: "G/5"
