File: bbb-parallel-cape.sch (KiCad schematic (older format))
At the start: 20 parts, among them J101 DB25, J102 DB25, P101 IDC26, P102 BeagleBone_Black_Header, P103 BeagleBone_Black_Header, P104 IDC26, P105 Conn_02x03_Odd_Even, Q101 2N7002K, SW101 SW_Push, SW102 SW_Push

Commit message: revision1 files
Parts:
- removed J101: DB25, symbol DB25
- added J101: DB25F, symbol DB25F
- added Z105: GENERIC_BLOCK, symbol GENERIC_BLOCK
- J102: value DB25 -> DB25M
- Z101, Z103: PartNo 1175-1625-ND -> 1175-1444-ND
- renumbered Z105 to Z106
Connections:
- net GNDD: now also J101.18, J101.19, J101.20, J101.21
- net GND_OR_5V: now also J101.22, J101.23, J101.24, J101.25
- net IO0: now also J101.1
- net IO1: now also J101.14
- net IO10: now also J101.7
- net IO11: now also J101.8
- net IO12: now also J101.9
- net IO13: now also J101.10
- net IO14: now also J101.11
- net IO15: now also J101.12
- net IO16: now also J101.13
- net IO2: now also J101.2
- net IO3: now also J101.15
- net IO4: now also J101.3
- net IO5: now also J101.16
- net IO6: now also J101.4
- net IO7: now also J101.17
- net IO8: now also J101.5
- net IO9: now also J101.6
Other:
- note added: "External \nPower Button"

Commit message: revision 1.1 before via stitching
Connections:
- net +3V3: now also JP101.6
- net GNDD: no longer JP101.6
- net PU_OR_PD renamed PULLUP_REF
Changed lines of the file:
@@
 Title "BeagleBone Parallel Port Cape"
 Date ""
-Rev "1"
-Comp "Rössler Systems"
+Rev "1.1"
+Comp "Machine Koder"
 Comment1 ""
 Comment2 ""
@@
 $EndComp
 Text GLabel 2050 6100 2    50   UnSpc ~ 0
-PU_OR_PD
+PULLUP_REF
 $Comp
 L GNDD #PWR017
 U 1 1 5A30FF02
-P 1650 6550
-F 0 "#PWR017" H 1650 6300 50  0001 C CNN
-F 1 "GNDD" H 1650 6400 50  0000 C CNN
-F 2 "" H 1650 6550 60  0000 C CNN
-F 3 "" H 1650 6550 60  0000 C CNN
-	1    1650 6550
+P 1550 6550
+F 0 "#PWR017" H 1550 6300 50  0001 C CNN
+F 1 "GNDD" H 1550 6400 50  0000 C CNN
+F 2 "" H 1550 6550 60  0000 C CNN
+F 3 "" H 1550 6550 60  0000 C CNN
+	1    1550 6550
 	1    0    0    -1
 $EndComp
@@
 Connection ~ 1650 5750
 Wire Wire Line
-	1550 6350 1550 6450
-Wire Wire Line
-	1550 6450 1750 6450
-Wire Wire Line
-	1750 6450 1750 6350
-Wire Wire Line
-	1650 6450 1650 6550
-Connection ~ 1650 6450
-Wire Wire Line
 	1300 6100 1450 6100
 Wire Wire Line
@@
 	1    0    0    -1
 $EndComp
+Wire Wire Line
+	1550 6350 1550 6550
+$Comp
+L +3V3 #PWR?
+U 1 1 5A9CB293
+P 2000 6550
+F 0 "#PWR?" H 2000 6400 50  0001 C CNN
+F 1 "+3V3" H 2000 6690 50  0000 C CNN
+F 2 "" H 2000 6550 60  0000 C CNN
+F 3 "" H 2000 6550 60  0000 C CNN
+	1    2000 6550
+	1    0    0    -1
+$EndComp
+Wire Wire Line
+	1750 6650 2000 6650
+Wire Wire Line
+	2000 6650 2000 6550
+Wire Wire Line
+	1750 6350 1750 6650
 $EndSCHEMATC

Commit message: updating project
Parts:
- added Z107, Z108: GENERIC_BLOCK, symbol GENERIC_BLOCK
- J101: AssemblyVariant (none) -> 3; Mfg (none) -> CNC Tech; PartNo (none) -> 410F0-25-1-00
- J102, Z103, Z104: AssemblyVariant 2 -> 3
- Q101: Mfg Diodes Inc. -> ON Semiconductor; PartNo 2N7002K-7DICT-ND -> 2N7002KT1GOSCT-ND
- Z101, Z102: AssemblyVariant 1 -> 3
Other:
- note added: "Jumper\nShorting"
Changed lines of the file:
@@
 F 4 "1175-1815-ND" H 10350 5000 60  0001 C CNN "PartNo"
 F 5 "CNC Tech" H 10350 5000 60  0001 C CNN "Mfg"
-F 6 "2" H 10350 5000 60  0001 C CNN "AssemblyVariant"
+F 6 "3" H 10350 5000 60  0001 C CNN "AssemblyVariant"
 	1    10350 5000
 	1    0    0    -1
@@
 F 2 "2N7002K-7:SOT95P240X105-3N" H 5700 6550 50  0001 C CNN
 F 3 "" H 5500 6450 50  0000 C CNN
-F 4 "2N7002K-7DICT-ND" H 5500 6450 60  0001 C CNN "PartNo"
-F 5 "Diodes Inc." H 5500 6450 60  0001 C CNN "Mfg"
+F 4 "2N7002KT1GOSCT-ND" H 5500 6450 60  0001 C CNN "PartNo"
+F 5 "ON Semiconductor" H 5500 6450 60  0001 C CNN "Mfg"
 F 6 "1" H 5500 6450 60  0001 C CNN "AssemblyVariant"
 	1    5500 6450
@@
 F 4 "1175-1444-ND" H 7500 2800 60  0001 C CNN "PartNo"
 F 5 "CNC Tech" H 7500 2800 60  0001 C CNN "Mfg"
-F 6 "1" H 7500 2800 60  0001 C CNN "AssemblyVariant"
+F 6 "3" H 7500 2800 60  0001 C CNN "AssemblyVariant"
 	1    7500 2800
 	1    0    0    -1
@@
 F 4 "MC26G-5-ND" H 8300 2800 60  0001 C CNN "PartNo"
 F 5 "3M" H 8300 2800 60  0001 C CNN "Mfg"
-F 6 "1" H 8300 2800 60  0001 C CNN "AssemblyVariant"
+F 6 "3" H 8300 2800 60  0001 C CNN "AssemblyVariant"
 	1    8300 2800
 	1    0    0    -1
@@
 F 4 "1175-1444-ND" H 7500 5700 60  0001 C CNN "PartNo"
 F 5 "CNC Tech" H 7500 5700 60  0001 C CNN "Mfg"
-F 6 "2" H 7500 5700 60  0001 C CNN "AssemblyVariant"
+F 6 "3" H 7500 5700 60  0001 C CNN "AssemblyVariant"
 	1    7500 5700
 	1    0    0    -1
@@
 F 4 "MC26G-5-ND" H 8300 5700 60  0001 C CNN "PartNo"
 F 5 "3M" H 8300 5700 60  0001 C CNN "Mfg"
-F 6 "2" H 8300 5700 60  0001 C CNN "AssemblyVariant"
+F 6 "3" H 8300 5700 60  0001 C CNN "AssemblyVariant"
 	1    8300 5700
 	1    0    0    -1
@@
 F 2 "" H 10350 2100 50  0000 C CNN
 F 3 "" H 10350 2100 50  0000 C CNN
+F 4 "410F0-25-1-00" H 10350 2100 60  0001 C CNN "PartNo"
+F 5 "CNC Tech" H 10350 2100 60  0001 C CNN "Mfg"
+F 6 "3" H 10350 2100 60  0001 C CNN "AssemblyVariant"
 	1    10350 2100
 	1    0    0    -1
@@
 	1550 6350 1550 6550
 $Comp
-L +3V3 #PWR?
+L +3V3 #PWR040
 U 1 1 5A9CB293
 P 2000 6550
-F 0 "#PWR?" H 2000 6400 50  0001 C CNN
+F 0 "#PWR040" H 2000 6400 50  0001 C CNN
 F 1 "+3V3" H 2000 6690 50  0000 C CNN
 F 2 "" H 2000 6550 60  0000 C CNN
@@
 Wire Wire Line
 	1750 6350 1750 6650
+$Comp
+L GENERIC_BLOCK Z107
+U 1 1 5AC3EAF1
+P 1250 7250
+F 0 "Z107" H 1500 7550 60  0000 C CNN
+F 1 "GENERIC_BLOCK" H 1250 6900 60  0001 C CNN
+F 2 "" H 1250 7250 60  0001 C CNN
+F 3 "" H 1250 7250 60  0001 C CNN
+F 4 "S9000-ND" H 1250 7250 60  0001 C CNN "PartNo"
+F 5 "Sullins" H 1250 7250 60  0001 C CNN "Mfg"
+F 6 "1" H 1250 7250 60  0001 C CNN "AssemblyVariant"
+	1    1250 7250
+	1    0    0    -1
+$EndComp
+Text Notes 1050 7350 0    60   ~ 0
+Jumper\nShorting
+$Comp
+L GENERIC_BLOCK Z108
+U 1 1 5AC3F0D0
+P 2050 7250
+F 0 "Z108" H 2300 7550 60  0000 C CNN
+F 1 "GENERIC_BLOCK" H 2050 6900 60  0001 C CNN
+F 2 "" H 2050 7250 60  0001 C CNN
+F 3 "" H 2050 7250 60  0001 C CNN
+F 4 "S9000-ND" H 2050 7250 60  0001 C CNN "PartNo"
+F 5 "Sullins" H 2050 7250 60  0001 C CNN "Mfg"
+F 6 "1" H 2050 7250 60  0001 C CNN "AssemblyVariant"
+	1    2050 7250
+	1    0    0    -1
+$EndComp
+Text Notes 1850 7350 0    60   ~ 0
+Jumper\nShorting
 $EndSCHEMATC
